File: hardware/designs/KiCad/ShotTimer/ShotTimer.kicad_pcb (KiCad board)
At the start: 2 copper layers, 0 parts

Commit message: Rev 1.1 - optimized parts, updated BOM, reorged kicad part deps, started PCB layout
Parts:
- added BZ1: Speaker, ShotTimer:PS1420P02CT, F.Cu at (259.1, -21.6)
- added C1: 10uF, Capacitor_THT:C_Disc_D4.7mm_W2.5mm_P5.00mm, F.Cu at (67.0, -62.1)
- added C10: 10uF, Capacitor_THT:C_Disc_D4.7mm_W2.5mm_P5.00mm, F.Cu at (55.7, -67.5)
- added C13: 0.1uF, Capacitor_THT:C_Disc_D5.1mm_W3.2mm_P5.00mm, F.Cu at (50.4, -67.5)
- added C14: 0.1uF, Capacitor_THT:C_Disc_D5.1mm_W3.2mm_P5.00mm, F.Cu at (-175.5, 116.8)
- added C15: 22pF, Capacitor_THT:C_Disc_D3.8mm_W2.6mm_P2.50mm, F.Cu at (42.8, -76.4)
- added C16: 22pF, Capacitor_THT:C_Disc_D3.8mm_W2.6mm_P2.50mm, F.Cu at (37.9, -76.4)
- added C17: 0.1uF, Capacitor_THT:C_Disc_D5.1mm_W3.2mm_P5.00mm, F.Cu at (164.9, 275.7)
- added C18: 10uF, Capacitor_THT:C_Disc_D4.7mm_W2.5mm_P5.00mm, F.Cu at (-175.1, 107.1)
- added C19: 10uF, Capacitor_THT:C_Disc_D4.7mm_W2.5mm_P5.00mm, F.Cu at (178.9, 269.0)
- added C2: 10uF, Capacitor_THT:C_Disc_D4.7mm_W2.5mm_P5.00mm, F.Cu at (26.4, -114.2)
- added C20: 10uF, Capacitor_THT:C_Disc_D4.7mm_W2.5mm_P5.00mm, F.Cu at (77.9, -144.3)
- added C21: 0.1uF, Capacitor_THT:C_Disc_D5.1mm_W3.2mm_P5.00mm, F.Cu at (72.4, -144.3)
- added C22: 0.1uF, Capacitor_THT:C_Disc_D5.1mm_W3.2mm_P5.00mm, F.Cu at (-169.5, -90.4)
- added C23: 10nF, Capacitor_THT:C_Disc_D4.7mm_W2.5mm_P5.00mm, F.Cu at (-165.6, -101.5)
- added C24: 1uF, Capacitor_THT:C_Disc_D7.5mm_W4.4mm_P5.00mm, F.Cu at (-173.3, -113.6)
- added C25: 100pF, Capacitor_THT:C_Disc_D3.8mm_W2.6mm_P2.50mm, F.Cu at (-169.0, -126.3)
- added C26: 0.1uF, Capacitor_THT:C_Disc_D5.1mm_W3.2mm_P5.00mm, F.Cu at (-215.7, -115.6)
- added C27: 10uF, Capacitor_THT:C_Disc_D4.7mm_W2.5mm_P5.00mm, F.Cu at (-194.9, -124.5)
- added C3: 0.1uF, Capacitor_THT:C_Disc_D5.1mm_W3.2mm_P5.00mm, F.Cu at (32.2, -114.2)
- added C4: 0.1uF, Capacitor_THT:C_Disc_D5.1mm_W3.2mm_P5.00mm, F.Cu at (72.3, -62.1)
- added C5: 220uF, Capacitor_THT:CP_Radial_D8.0mm_P3.50mm, F.Cu at (309.2, -34.0)
- added C6: 220uF, Capacitor_THT:CP_Radial_D8.0mm_P3.50mm, F.Cu at (90.3, -50.5)
- added C7: 220uF, Capacitor_THT:CP_Radial_D8.0mm_P3.50mm, F.Cu at (319.9, -34.0)
- added C8: 10uF, Capacitor_THT:C_Disc_D4.7mm_W2.5mm_P5.00mm, F.Cu at (267.8, -15.6)
- added C9: 0.1uF, Capacitor_THT:C_Disc_D5.1mm_W3.2mm_P5.00mm, F.Cu at (267.8, -21.6)
- added D1: 1N5817, Diode_THT:D_DO-41_SOD81_P10.16mm_Horizontal, F.Cu at (71.8, -115.5)
- added D10: 1N5817, Diode_THT:D_DO-41_SOD81_P10.16mm_Horizontal, F.Cu at (301.1, -31.5)
- added D11: 1N5817, Diode_THT:D_DO-41_SOD81_P10.16mm_Horizontal, F.Cu at (301.1, -36.6)
- added D2: 1N5817, Diode_THT:D_DO-41_SOD81_P10.16mm_Horizontal, F.Cu at (61.7, -115.5)
- added D3: 1N5817, Diode_THT:D_DO-41_SOD81_P10.16mm_Horizontal, F.Cu at (76.9, -115.6)
- added D4: 1N5817, Diode_THT:D_DO-41_SOD81_P10.16mm_Horizontal, F.Cu at (82.0, -115.6)
- added D5: 1N5817, Diode_THT:D_DO-41_SOD81_P10.16mm_Horizontal, F.Cu at (66.8, -115.6)
- added D6: 1N5817, Diode_THT:D_DO-41_SOD81_P10.16mm_Horizontal, F.Cu at (87.0, -115.5)
- added D7: 1N5817, Diode_THT:D_DO-41_SOD81_P10.16mm_Horizontal, F.Cu at (92.1, -115.5)
- added D8: 1N5817, Diode_THT:D_DO-41_SOD81_P10.16mm_Horizontal, F.Cu at (97.2, -115.5)
- added D9: 1N5817, Diode_THT:D_DO-41_SOD81_P10.16mm_Horizontal, F.Cu at (327.5, -33.0)
- added DS1: NHD-0420CW-SPI, NHD_NHD-0420CW-AG3, F.Cu at (51.8, -232.0)
- added FB1: Ferrite_Bead, Ferrite_THT:LairdTech_28C0236-0JW-10, F.Cu at (-81.7, -39.3)
- added FB2: Ferrite_Bead, Ferrite_THT:LairdTech_28C0236-0JW-10, F.Cu at (-90.3, -35.5)
- added J1: SYS_PWR, TerminalBlock:TerminalBlock_bornier-2_P5.08mm, F.Cu at (340.4, -16.5)
- added J2: ISP, Connector_PinHeader_2.54mm:PinHeader_2x03_P2.54mm_Vertical, F.Cu at (294.0, -17.8)
- added J3: SERIAL, Connector_PinHeader_2.54mm:PinHeader_1x02_P2.54mm_Vertical, F.Cu at (280.0, -16.5)
- added J4: Conn_01x20, Connector_PinSocket_2.54mm:PinSocket_1x20_P2.54mm_Vertical, F.Cu at (74.9, -148.2)
- added J5: Conn_01x20, Connector_PinHeader_2.54mm:PinHeader_1x20_P2.54mm_Vertical, F.Cu at (76.1, -251.7)
- added JP1: SYS_CFG, Connector_PinHeader_2.54mm:PinHeader_1x02_P2.54mm_Vertical, F.Cu at (67.0, -51.0)
- added JP2: ISP_PWR, Connector_PinHeader_2.54mm:PinHeader_1x03_P2.54mm_Vertical, F.Cu at (300.6, -15.2)
- added L1: 33uH, Inductor_THT:L_Radial_D7.8mm_P5.00mm_Fastron_07HCP, F.Cu at (319.4, -29.0)
- added LED1: Green, LED_THT:LED_D3.0mm, F.Cu at (5.77, -100.3)
- added LED2: Yellow, LED_THT:LED_D3.0mm, F.Cu at (19.0, -100.6)
- added LED3: Red, LED_THT:LED_D3.0mm, F.Cu at (32.3, -100.5)
- added LED4: Yellow, LED_THT:LED_D3.0mm, F.Cu at (45.6, -100.5)
- added MK1: CMA-4544PF-W, MIC_CMA-4544PF-W, F.Cu at (-200.1, -96.1)
- added Q1: Q_NPN_EBC, Package_TO_SOT_THT:TO-92, F.Cu at (256.4, -34.8)
- added Q2: Q_PNP_CBE, Package_TO_SOT_THT:TO-92, F.Cu at (296.0, -22.9)
- added R1: 10K, Resistor_THT:R_Axial_DIN0207_L6.3mm_D2.5mm_P7.62mm_Horizontal, F.Cu at (72.3, -44.1)
- added R10: 10K, Resistor_THT:R_Axial_DIN0207_L6.3mm_D2.5mm_P7.62mm_Horizontal, F.Cu at (82.0, -91.4)
- added R11: 10K, Resistor_THT:R_Axial_DIN0207_L6.3mm_D2.5mm_P7.62mm_Horizontal, F.Cu at (66.8, -91.4)
- added R12: 10K, Resistor_THT:R_Axial_DIN0207_L6.3mm_D2.5mm_P7.62mm_Horizontal, F.Cu at (87.0, -91.4)
- added R13: 10K, Resistor_THT:R_Axial_DIN0207_L6.3mm_D2.5mm_P7.62mm_Horizontal, F.Cu at (92.1, -91.4)
- added R14: 10K, Resistor_THT:R_Axial_DIN0207_L6.3mm_D2.5mm_P7.62mm_Horizontal, F.Cu at (97.2, -91.4)
- added R15: 100K, Resistor_THT:R_Axial_DIN0207_L6.3mm_D2.5mm_P7.62mm_Horizontal, F.Cu at (375.5, -6.55)
- added R16: 10K, Resistor_THT:R_Axial_DIN0207_L6.3mm_D2.5mm_P7.62mm_Horizontal, F.Cu at (267.8, -33.5)
- added R17: 1K, Resistor_THT:R_Axial_DIN0207_L6.3mm_D2.5mm_P7.62mm_Horizontal, F.Cu at (275.5, -27.9)
- added R18: 10K, Resistor_THT:R_Axial_DIN0207_L6.3mm_D2.5mm_P7.62mm_Horizontal, F.Cu at (20.6, -5.91)
- added R19: 10K, Resistor_THT:R_Axial_DIN0207_L6.3mm_D2.5mm_P7.62mm_Horizontal, F.Cu at (304.7, -27.6)
- added R2: 10K, Resistor_THT:R_Axial_DIN0207_L6.3mm_D2.5mm_P7.62mm_Horizontal, F.Cu at (82.9, -51.8)
- added R20: 10K, Resistor_THT:R_Axial_DIN0207_L6.3mm_D2.5mm_P7.62mm_Horizontal, F.Cu at (312.3, -22.5)
- added R21: 330, Resistor_THT:R_Axial_DIN0204_L3.6mm_D1.6mm_P5.08mm_Horizontal, F.Cu at (5.77, -91.3)
- added R22: 330, Resistor_THT:R_Axial_DIN0204_L3.6mm_D1.6mm_P5.08mm_Horizontal, F.Cu at (19.0, -91.3)
- added R23: 330, Resistor_THT:R_Axial_DIN0204_L3.6mm_D1.6mm_P5.08mm_Horizontal, F.Cu at (32.3, -91.3)
- added R24: 330, Resistor_THT:R_Axial_DIN0204_L3.6mm_D1.6mm_P5.08mm_Horizontal, F.Cu at (45.6, -91.3)
- added R25: 10K, Resistor_THT:R_Axial_DIN0207_L6.3mm_D2.5mm_P7.62mm_Horizontal, F.Cu at (141.0, 261.5)
- added R26: 10K, Resistor_THT:R_Axial_DIN0207_L6.3mm_D2.5mm_P7.62mm_Horizontal, F.Cu at (154.0, 266.5)
- added R27: 10K, Resistor_THT:R_Axial_DIN0207_L6.3mm_D2.5mm_P7.62mm_Horizontal, F.Cu at (162.2, 258.0)
- added R28: 10K, Resistor_THT:R_Axial_DIN0207_L6.3mm_D2.5mm_P7.62mm_Horizontal, F.Cu at (-162.5, 113.4)
- added R29: 2K, Resistor_THT:R_Axial_DIN0207_L6.3mm_D2.5mm_P7.62mm_Horizontal, F.Cu at (-185.3, -99.6)
- added R3: 10K, Resistor_THT:R_Axial_DIN0207_L6.3mm_D2.5mm_P7.62mm_Horizontal, F.Cu at (77.6, -51.8)
- added R30: 2K, Resistor_THT:R_Axial_DIN0207_L6.3mm_D2.5mm_P7.62mm_Horizontal, F.Cu at (-191.3, -86.1)
- added R31: 10K, Resistor_THT:R_Axial_DIN0207_L6.3mm_D2.5mm_P7.62mm_Horizontal, F.Cu at (36.8, -144.3)
- added R32: 10K, Resistor_THT:R_Axial_DIN0207_L6.3mm_D2.5mm_P7.62mm_Horizontal, F.Cu at (31.8, -136.7)
- added R33: 1M, Resistor_THT:R_Axial_DIN0207_L6.3mm_D2.5mm_P7.62mm_Horizontal, F.Cu at (-153.6, -96.6)
- added R34: 1M, Resistor_THT:R_Axial_DIN0207_L6.3mm_D2.5mm_P7.62mm_Horizontal, F.Cu at (-147.9, -83.2)
- added R35: 10K, Resistor_THT:R_Axial_DIN0207_L6.3mm_D2.5mm_P7.62mm_Horizontal, F.Cu at (64.8, -136.7)
- added R36: 10K, Resistor_THT:R_Axial_DIN0207_L6.3mm_D2.5mm_P7.62mm_Horizontal, F.Cu at (47.0, -136.7)
- added R37: 10K, Resistor_THT:R_Axial_DIN0207_L6.3mm_D2.5mm_P7.62mm_Horizontal, F.Cu at (-191.7, -110.8)
- added R38: 100K, Resistor_THT:R_Axial_DIN0207_L6.3mm_D2.5mm_P7.62mm_Horizontal, F.Cu at (-136.1, -109.7)
- added R39: 10K, Resistor_THT:R_Axial_DIN0207_L6.3mm_D2.5mm_P7.62mm_Horizontal, F.Cu at (56.7, -91.4)
- added R4: 316K 1%, Resistor_THT:R_Axial_DIN0207_L6.3mm_D2.5mm_P7.62mm_Horizontal, F.Cu at (304.8, -17.1)
- added R5: 412K 1%, Resistor_THT:R_Axial_DIN0207_L6.3mm_D2.5mm_P7.62mm_Horizontal, F.Cu at (354.1, -3.20)
- added R6: 10K, Resistor_THT:R_Axial_DIN0207_L6.3mm_D2.5mm_P7.62mm_Horizontal, F.Cu at (364.2, -17.2)
- added R7: 10K, Resistor_THT:R_Axial_DIN0207_L6.3mm_D2.5mm_P7.62mm_Horizontal, F.Cu at (71.8, -91.4)
- added R8: 10K, Resistor_THT:R_Axial_DIN0207_L6.3mm_D2.5mm_P7.62mm_Horizontal, F.Cu at (61.7, -91.4)
- added R9: 10K, Resistor_THT:R_Axial_DIN0207_L6.3mm_D2.5mm_P7.62mm_Horizontal, F.Cu at (76.9, -91.4)
- added SW1: BTN, ShotTimer:SW_B3F-10xx, F.Cu at (19.2, -74.2)
- added SW2: BTN, ShotTimer:SW_B3F-10xx, F.Cu at (19.2, -83.8)
- added SW3: BTN, ShotTimer:SW_B3F-10xx, F.Cu at (28.9, -74.2)
- added SW4: BTN, ShotTimer:SW_B3F-10xx, F.Cu at (19.2, -64.5)
- added SW5: BTN, ShotTimer:SW_B3F-10xx, F.Cu at (9.58, -74.2)
- added SW6: BTN, ShotTimer:SW_B3F-10xx, F.Cu at (56.5, -83.1)
- added SW7: BTN, ShotTimer:SW_B3F-10xx, F.Cu at (75.2, -83.1)
- added SW8: BTN, ShotTimer:SW_B3F-10xx, F.Cu at (94.0, -83.1)
- added SW9: Reset, ShotTimer:SW_B3F-10xx, F.Cu at (10.7, -8.51)
- added U1: CD74HC151E, Package_DIP:DIP-16_W7.62mm, F.Cu at (39.0, -106.6)
- added U2: TSR_1-2433, Converter_DCDC:Converter_DCDC_TRACO_TSR-1_THT, F.Cu at (78.9, -62.1)
- added U3: RN4871-I/RM140, RF_Module:Microchip_RN4871, F.Cu at (92.3, -60.5)
- added U4: LT1303CN8-5#PBF, ShotTimer:PDIP-8_N, F.Cu at (324.5, -20.3)
- added U5: ATmega328P-PU, Package_DIP:DIP-28_W7.62mm, F.Cu at (62.0, -62.7)
- added U6: MCP3201, Package_DIP:DIP-8_W7.62mm, F.Cu at (-165.1, 129.8)
- added U7: 25LC1024-I/P, Package_DIP:DIP-8_W7.62mm, F.Cu at (145.6, 275.0)
- added U8: MAX4466EXK, SOT65P210X110-5N, F.Cu at (-152.5, -116.7)
- added Y1: 16MHz, Crystal:Crystal_HC49-U_Vertical, F.Cu at (42.8, -69.2)
Routing:
- net Net-(D4-Pad2): track 0.00 -> 123.4 mm
- net Net-(D3-Pad2): track 0.00 -> 101.6 mm
- net Net-(D1-Pad2): track 0.00 -> 98.1 mm
- net Net-(D5-Pad2): track 0.00 -> 94.5 mm
- net Net-(D6-Pad2): track 0.00 -> 87.4 mm
- net +5V: track 0.00 -> 84.2 mm
- net Net-(D7-Pad2): track 0.00 -> 74.9 mm
- net Net-(D8-Pad2): track 0.00 -> 72.9 mm
- net Net-(D2-Pad2): track 0.00 -> 67.7 mm
- net BUTTON_PUSHED: track 0.00 -> 35.6 mm
- net TX: track 0.00 -> 34.2 mm
- net Net-(D10-Pad2): track 0.00 -> 33.7 mm
- net RX: track 0.00 -> 31.5 mm
- net PWR: track 0.00 -> 25.5 mm
- net Net-(BZ1-Pad2): track 0.00 -> 24.9 mm
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Other:
- board outline added: 351.2 x 152.4 mm
- net class Default: clearance 0.2 -> 0.254; trace_width 0.25 -> 0.1524; via_dia 0.8 -> 0.508; via_drill 0.4 -> 0.254
- rule pad_to_mask_clearance: 0 -> 0.0508
- rule trace_clearance: 0.2 -> 0.254
- rule via_min_drill: 0.3 -> 0.254
- rule via_min_size: 0.0254 -> 0.508
- board text added: "ACT"
- board text added: "LOW"
- board text added: "PGML1"
- board text added: "PWR"

Commit message: initial pcb layout, bump to rev 1.2 remove 10uF caps, tidy up
Parts:
- removed C10, C18, C19, C20, C27, C8: 10uF, Capacitor_THT:C_Disc_D4.7mm_W2.5mm_P5.00mm
- C1, C2: value 10uF -> 0.1uF; footprint Capacitor_THT:C_Disc_D4.7mm_W2.5mm_P5.00mm -> Capacitor_THT:C_Disc_D5.1mm_W3.2mm_P5.00mm
- moved C17 371.1 mm to (38.7, -73.2), turned to 270 degrees
- moved R26 358.1 mm to (49.3, -76.0), turned to 270 degrees
- moved U7 348.8 mm to (38.7, -57.0), turned to 90 degrees
- moved R25 348.3 mm to (54.8, -76.0), turned to 270 degrees
- moved R27 347.0 mm to (43.9, -68.2), turned to 90 degrees
- moved R15 283.5 mm to (92.1, -14.5), turned to 90 degrees
- moved R5 275.4 mm to (81.0, -38.5), turned to 90 degrees
- moved R6 267.3 mm to (96.9, -14.5), turned to 90 degrees
- moved C26 262.9 mm to (27.9, -16.9), turned to 90 degrees
- moved C14 259.1 mm to (43.0, -22.4), turned to 270 degrees
- moved U6 258.7 mm to (48.5, -16.1), turned to 90 degrees
- moved J1 248.4 mm to (92.1, -6.16)
- moved R28 242.8 mm to (37.9, -23.7), turned to 270 degrees
- moved D9 241.8 mm to (86.2, -48.9)
- moved R37 238.6 mm to (25.7, -12.4), turned to 270 degrees
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Connections:
- net /VCC renamed /ISP_PWR
- C1 pad 1: +5V -> GND
- C1 pad 2: GND -> Net-(C1-Pad2)
- C17 pad 1: +5V -> GND
- C17 pad 2: GND -> +5V
- C2 pad 1: +5V -> GND
- C2 pad 2: GND -> +5V
- C6 pad 1: Net-(C6-Pad1) -> Net-(C1-Pad2)
- C9 pad 1: +5V -> GND
- C9 pad 2: GND -> +5V
- U2 pad 3: Net-(C6-Pad1) -> Net-(C1-Pad2)
- U3 pad 14: Net-(C6-Pad1) -> Net-(C1-Pad2)
- U5 pad 11: S1 -> ACTIVITY
- U5 pad 12: S2 -> PGML1
- U5 pad 13: Write_Protection -> PGM_RF
- U5 pad 14: SS_EEPROM -> SPEAKER_PWM
- U5 pad 15: SS_DS -> SS_EEPROM
- U5 pad 16: SS_ADC -> Write_Protection
- U5 pad 23: ACTIVITY -> BUTTON_PUSHED
- U5 pad 24: MIC_AMP_OUT -> S2
- U5 pad 25: PGML1 -> S1
- U5 pad 26: BUTTON_PUSHED -> S0
- U5 pad 27: PGM_RF -> Y
- U5 pad 28: SPEAKER_PWM -> ~Y
- U5 pad 4: Y -> SS_ADC
- U5 pad 5: ~Y -> SS_DS
- U5 pad 6: S0 -> Net-(U5-Pad6)
Routing:
- net SCK: track 0.00 -> 283.2 mm, vias 0 -> 1
- net MISO: track 0.00 -> 278.1 mm, vias 0 -> 1
- net MOSI: track 0.00 -> 275.5 mm, vias 0 -> 1
- net ISP_RESET: track 14.3 -> 216.1 mm, vias 0 -> 1
- net RX: track 31.5 -> 204.0 mm, vias 0 -> 1
- net TX: track 34.2 -> 197.4 mm, vias 0 -> 1
- net SS_DS: track 0.00 -> 144.5 mm
- net BUTTON_PUSHED: track 35.6 -> 172.4 mm
- net S2: track 0.00 -> 127.9 mm
- net LBO: track 0.00 -> 123.5 mm, vias 0 -> 1
- net S1: track 0.00 -> 120.9 mm
- net S0: track 0.00 -> 113.9 mm
- net Y: track 0.00 -> 101.6 mm, vias 0 -> 1
- net ~Y: track 0.00 -> 99.5 mm, vias 0 -> 1
- net SS_ADC: track 0.00 -> 93.6 mm
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- added copper zone on F.Cu, net +5V
- added copper zone on F.Cu, net +5VA
- added copper zone on B.Cu, net GND
- added copper zone on B.Cu, net GNDA
Other:
- board size 351.2 x 152.4 mm -> 101.6 x 152.4 mm
- net class Default: clearance 0.254 -> 0.2032
- rule trace_clearance: 0.254 -> 0.2032
- board text added: "Jason Sipula"
- board text added: "March 6, 2021"
- board text added: "REV 1.2"
- board text added: "Shot Timer"
- board text removed: "ACT"
- board text removed: "LOW"
- board text removed: "PGML1"
- board text removed: "PWR"

Commit message: PCB REV1.3 - first design sent to fab.
Parts:
- removed J4: Conn_01x20, Connector_PinSocket_2.54mm:PinSocket_1x20_P2.54mm_Vertical
- removed J5: Conn_01x20, Connector_PinHeader_2.54mm:PinHeader_1x20_P2.54mm_Vertical
- DS1: footprint NHD_NHD-0420CW-AG3 -> ShotTimer:NHD_NHD-0420CW-AG3
- moved DS1 286.7 mm to (84.8, 47.4)
- moved C1 184.5 mm to (127.3, 133.7)
- moved C6 184.5 mm to (99.0, 119.7)
- moved C7 184.5 mm to (116.9, 151.6)
- moved D6 184.5 mm to (121.0, 65.9)
- moved D8 184.5 mm to (131.1, 65.9)
- moved J1 184.5 mm to (126.1, 175.2)
- moved R20 184.5 mm to (113.7, 172.7)
- moved R35 184.5 mm to (98.7, 44.7)
- moved R5 184.5 mm to (115.0, 142.9)
- moved C17 184.5 mm to (72.6, 108.1)
- moved C2 184.5 mm to (65.4, 124.0)
- moved C3 184.5 mm to (66.1, 67.1)
- moved D1 184.5 mm to (105.8, 65.8)
- moved D10 184.5 mm to (102.9, 158.2)
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Connections:
- DS1 pad 1: Net-(DS1-Pad1) -> GND
- DS1 pad 11: Net-(DS1-Pad11) -> Net-(DS1-Pad10)
- DS1 pad 12: Net-(DS1-Pad12) -> Net-(DS1-Pad10)
- DS1 pad 13: Net-(DS1-Pad13) -> Net-(DS1-Pad10)
- DS1 pad 14: Net-(DS1-Pad14) -> Net-(DS1-Pad10)
- DS1 pad 15: Net-(DS1-Pad15) -> SS_DS
- DS1 pad 18: Net-(DS1-Pad18) -> Net-(DS1-Pad17)
- DS1 pad 19: Net-(DS1-Pad19) -> Net-(DS1-Pad17)
- DS1 pad 2: Net-(DS1-Pad2) -> +5V
- DS1 pad 20: Net-(DS1-Pad20) -> GND
- DS1 pad 3: Net-(DS1-Pad3) -> +5V
- DS1 pad 5: Net-(DS1-Pad5) -> Net-(DS1-Pad4)
- DS1 pad 6: Net-(DS1-Pad6) -> Net-(DS1-Pad4)
- DS1 pad 7: Net-(DS1-Pad7) -> SCK
- DS1 pad 8: Net-(DS1-Pad8) -> MOSI
- DS1 pad 9: Net-(DS1-Pad9) -> MISO
- R31 pad 1: Net-(J4-Pad16) -> Net-(DS1-Pad16)
- R32 pad 2: Net-(J4-Pad17) -> Net-(DS1-Pad17)
- R35 pad 2: Net-(J4-Pad4) -> Net-(DS1-Pad4)
- R36 pad 2: Net-(J4-Pad10) -> Net-(DS1-Pad10)
Routing:
- net Net-(J4-Pad10): track 14.1 -> 0.00 mm
- net Net-(DS1-Pad10): track 0.00 -> 14.1 mm
- net Net-(J4-Pad4): track 8.99 -> 0.00 mm
- net Net-(J4-Pad17): track 8.99 -> 0.00 mm
- net Net-(DS1-Pad4): track 0.00 -> 8.99 mm
- net Net-(DS1-Pad17): track 0.00 -> 8.99 mm
- net Net-(J4-Pad16): track 3.91 -> 0.00 mm
- net Net-(DS1-Pad16): track 0.00 -> 3.91 mm
- net GND: vias 4 -> 2
Other:
- board text added: "J4"
- board text added: "March 11, 2021"
- board text added: "REV 1.3"
- board text removed: "March 6, 2021"
- board text removed: "REV 1.2"
